File: PCB/RFfrontend.kicad_sch (KiCad schematic)
At the start: 0 parts

Commit message: what about actually comiting
Other:
- note added: "https://github.com/meshtastic/firmware/blob/develop/variants/stm32/rak3172/rfswitch.h"
Changed lines of the file:
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@@
 		(company "Tomas Kuchta")
+	)
+	(text "https://github.com/meshtastic/firmware/blob/develop/variants/stm32/rak3172/rfswitch.h"
+		(exclude_from_sim no)
+		(at 132.842 48.514 0)
+		(effects
+			(font
+				(size 1.27 1.27)
+			)
+		)
 	)
 	(text "BALFHB-WL-02D3\n\nMagic type ship"
