File: PCB/USBC.kicad_sch (KiCad schematic)
At the start: 4 parts, among them J1 UJ20-C-H-G-SMT-2A-P16-TR, U3 USBLC6-2SC6

Commit message: added the rak4630 module
Parts:
- renumbered R5 to R4, R4 to R5, U3 to U1
Changed lines of the file:
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@@
 		(dnp no)
 		(fields_autoplaced yes)
-		(property "Reference" "#PWR7"
+		(property "Reference" "#PWR07"
 			(at 63.5 119.38 0)
 			(hide yes)
@@
 		)
 		(instances
+			(project "USBC"
+				(path "/9402f0fd-4abf-4374-8b5f-14f4c6a25de3"
+					(reference "#PWR07")
+					(unit 1)
+				)
+			)
 			(project "UBS-C_TYPE-C-31-M-12"
 				(path "/d915b4b4-54fd-4193-8810-936621a064e8"
@@
 		(dnp no)
 		(fields_autoplaced yes)
-		(property "Reference" "U3"
+		(property "Reference" "U1"
 			(at 110.8711 77.47 0)
 			(show_name no)
@@
 		)
 		(instances
+			(project "USBC"
+				(path "/9402f0fd-4abf-4374-8b5f-14f4c6a25de3"
+					(reference "U1")
+					(unit 1)
+				)
+			)
 			(project "UBS-C_TYPE-C-31-M-12"
 				(path "/d915b4b4-54fd-4193-8810-936621a064e8"
@@
 		(dnp no)
 		(fields_autoplaced yes)
-		(property "Reference" "#PWR010"
+		(property "Reference" "#PWR02"
 			(at 109.22 81.28 0)
 			(hide yes)
@@
 		)
 		(instances
+			(project "USBC"
+				(path "/9402f0fd-4abf-4374-8b5f-14f4c6a25de3"
+					(reference "#PWR02")
+					(unit 1)
+				)
+			)
 			(project "UBS-C_TYPE-C-31-M-12"
 				(path "/d915b4b4-54fd-4193-8810-936621a064e8"
@@
 		)
 		(instances
+			(project "USBC"
+				(path "/9402f0fd-4abf-4374-8b5f-14f4c6a25de3"
+					(reference "#FLG01")
+					(unit 1)
+				)
+			)
 			(project "UBS-C_TYPE-C-31-M-12"
 				(path "/d915b4b4-54fd-4193-8810-936621a064e8"
@@
 		(in_pos_files yes)
 		(dnp no)
-		(property "Reference" "R5"
+		(property "Reference" "R4"
 			(at 97.79 100.3299 0)
 			(show_name no)
@@
 		)
 		(instances
+			(project "USBC"
+				(path "/9402f0fd-4abf-4374-8b5f-14f4c6a25de3"
+					(reference "R4")
+					(unit 1)
+				)
+			)
 			(project "UBS-C_TYPE-C-31-M-12"
 				(path "/d915b4b4-54fd-4193-8810-936621a064e8"
@@
 		(dnp no)
 		(fields_autoplaced yes)
-		(property "Reference" "#PWR08"
+		(property "Reference" "#PWR01"
 			(at 90.17 69.85 0)
 			(hide yes)
@@
 		)
 		(instances
+			(project "USBC"
+				(path "/9402f0fd-4abf-4374-8b5f-14f4c6a25de3"
+					(reference "#PWR01")
+					(unit 1)
+				)
+			)
 			(project "UBS-C_TYPE-C-31-M-12"
 				(path "/d915b4b4-54fd-4193-8810-936621a064e8"
@@
 		)
 		(instances
+			(project "USBC"
+				(path "/9402f0fd-4abf-4374-8b5f-14f4c6a25de3"
+					(reference "J1")
+					(unit 1)
+				)
+			)
 			(project "UBS-C_TYPE-C-31-M-12"
 				(path "/d915b4b4-54fd-4193-8810-936621a064e8"
@@
 		(dnp no)
 		(fields_autoplaced yes)
-		(property "Reference" "#PWR9"
+		(property "Reference" "#PWR08"
 			(at 92.71 116.84 0)
 			(hide yes)
@@
 		)
 		(instances
+			(project "USBC"
+				(path "/9402f0fd-4abf-4374-8b5f-14f4c6a25de3"
+					(reference "#PWR08")
+					(unit 1)
+				)
+			)
 			(project "UBS-C_TYPE-C-31-M-12"
 				(path "/d915b4b4-54fd-4193-8810-936621a064e8"
@@
 		(dnp no)
 		(fields_autoplaced yes)
-		(property "Reference" "#PWR15"
+		(property "Reference" "#PWR09"
 			(at 109.22 101.6 0)
 			(hide yes)
@@
 		)
 		(instances
+			(project "USBC"
+				(path "/9402f0fd-4abf-4374-8b5f-14f4c6a25de3"
+					(reference "#PWR09")
+					(unit 1)
+				)
+			)
 			(project "UBS-C_TYPE-C-31-M-12"
 				(path "/d915b4b4-54fd-4193-8810-936621a064e8"
@@
 		(in_pos_files yes)
 		(dnp no)
-		(property "Reference" "R4"
+		(property "Reference" "R5"
 			(at 87.63 100.3299 0)
 			(show_name no)
@@
 		)
 		(instances
+			(project "USBC"
+				(path "/9402f0fd-4abf-4374-8b5f-14f4c6a25de3"
+					(reference "R5")
+					(unit 1)
+				)
+			)
 			(project "UBS-C_TYPE-C-31-M-12"
 				(path "/d915b4b4-54fd-4193-8810-936621a064e8"
@@
 		)
 	)
+	(sheet_instances
+		(path "/"
+			(page "1")
+		)
+	)
+	(embedded_fonts no)
 )
