File: PCB/MCU.kicad_sch (KiCad schematic)
At the start: 9 parts, among them J1 UJ20-C-H-G-SMT-2A-P16-TR, J2 Conn_01x05_Pin, SW1 SKRKAHE020, U1 RAK4630, U2 USBLC6-2SC6

Commit message: a bit of polishing and work on the pheripherials
Parts:
- removed J1: UJ20-C-H-G-SMT-2A-P16-TR, Connector_USB:USB_C_Receptacle_HRO_TYPE-C-31-M-12, symbol Connector:USB_C_Receptacle_USB2.0_16P
- removed R4, R5: 0603 5k1, Resistor_SMD:R_0805_2012Metric_Pad1.20x1.40mm_HandSolder, symbol Device:R
- removed U2: USBLC6-2SC6, Package_TO_SOT_SMD:SOT-23-6, symbol Power_Protection:USBLC6-2SC6
- added J5: USB_C_Receptacle_USB2.0_16P, Connector_USB:USB_C_Receptacle_HRO_TYPE-C-31-M-12, symbol Connector:USB_C_Receptacle_USB2.0_16P
- added R10, R9: 5k1, Resistor_SMD:R_0805_2012Metric_Pad1.20x1.40mm_HandSolder, symbol Device:R
- added U7: USBLC6-2SC6, Package_TO_SOT_SMD:SOT-23-6, symbol Power_Protection:USBLC6-2SC6
- U1: Availability Not in stock -> (none); Check_prices https://www.snapeda.com/parts/RAK4630/RAK/view-part/?ref=eda -> (none); MF RAK -> (none); MP RAK4630 -> (none); MPN (none) -> RAK4630; Package Package -> (none); Price None -> (none)
Connections:
- net +3.3V is gone; now on net +3V3: R3.1
- net 3V3 is gone; now on net +3V3: J2.1 (Pin_1)
- net SWIO is gone; now on net SWDIO: U1.19 (SWDIO)
- net CC1: now also J5.A5 (CC1), R10.1
- net CC2: now also J5.B5 (CC2), R9.1
- net D+: now also J5.A6 (D+), J5.B6 (D+), U7.3 (I/O2)
- net D-: now also J5.A7 (D-), J5.B7 (D-), U7.1 (I/O1)
- net GNDREF: now also J5.A1 (GND), J5.A12 (GND), J5.B1 (GND), J5.B12 (GND), J5.SH (SHIELD), R10.2, R9.2, U7.2 (GND)
- net USB_D+: now also U7.4 (I/O2)
- net USB_D-: now also U7.6 (I/O1)
- net VBUS: now also J5.A4 (VBUS), J5.A9 (VBUS), J5.B4 (VBUS), J5.B9 (VBUS), U7.5 (VBUS)
- no-connect marks 9 -> 21
Other:
- sheet Pheripherials ports: added none; removed LED, RX, SCL, SDA, TX
- moved on the sheet: C1, J2, R3, SW1, U1
